File: EEG/EEG.kicad_pcb (KiCad board)
At the start: 4 copper layers, 100 x 50 mm, 47 parts, among them J1 USB_B_Micro, J2 Conn_01x08_Female, J3 Conn_01x08_Female, Q1 SS8050, Q2 SS8050, SW1 SW_Push, SW2 SW_Push, U1 AMS1117-3.3, U2 FT231XS, U3 ESP32-PICO-D4, U4 MAX7219

Commit message: just BOM and gerbers left
Parts:
- moved R5 4.28 mm to (114.8, 92.8)
- moved R6 1.80 mm to (114.6, 95.7)
Routing:
- net D-: track 11.2 -> 8.60 mm
- net Net-(R6-Pad1): track 3.91 -> 6.24 mm
- net Net-(R5-Pad1): track 4.77 -> 6.24 mm
- net D+: track 7.89 -> 8.68 mm, vias 2 -> 0
