File: EEG/EEG.kicad_pcb (KiCad board)
At the start: 4 copper layers, 100 x 50 mm, 47 parts, among them J1 USB_B_Micro, J2 Conn_01x08_Female, J3 Conn_01x08_Female, Q1 SS8050, Q2 SS8050, SW1 SW_Push, SW2 SW_Push, U1 AMS1117-3.3, U2 FT231XS, U3 ESP32-PICO-D4, U4 MAX7219

Commit message: generated gerbers
Parts:
- added G***: LOGO, logo:logo, F.Cu at (153.0, 68.6)
Other:
- board text removed: "Mohit Patel, Adam Schuhcknecht, Evan Fadanalli"
